Commit message: Completed urdf and added rviz config

File: pingpongbot_description/urdf/pingpongbot.urdf.xacro (robot description, xacro)
@@ -3,7 +3,7 @@
     <xacro:property name="yaml_dict" value="${xacro.load_yaml(params_yaml)['/**']['ros__parameters']}"/>
     <xacro:property name="wheel_radius" value="${yaml_dict['wheel_radius']}"/>
+    <xacro:property name="wheel_thickness" value="${yaml_dict['wheel_thickness']}"/>
     <xacro:property name="wheel_offset_radius" value="${yaml_dict['wheel_offset_radius']}"/>
-    <xacro:property name="bottom_base_height" value="${yaml_dict['bottom_base_height']}"/>
-    <xacro:property name="chassis_height" value="${yaml_dict['chassis_height']}"/>
+    <xacro:property name="origin_to_chassis_top" value="${yaml_dict['origin_to_chassis_top']}"/>
     <xacro:property name="paddle_origin_offset" value="${yaml_dict['paddle_origin_offset']}"/>
     <material name="white">
@@ -34,5 +34,5 @@
         <parent link="base_link"/>
         <child link="wheel1"/>
-        <origin xyz="${wheel_offset_radius} 0.0 0.0" rpy="0 1.57 0"/>
+        <origin xyz="0.0 ${-wheel_offset_radius} 0.0" rpy="${pi/2} 0 0"/>
         <axis xyz="0 0 1"/>
     </joint>
@@ -55,5 +55,5 @@
         <parent link="base_link"/>
         <child link="wheel2"/>
-        <origin xyz="${wheel_offset_radius} 0.0 0.0" rpy="-1.57 0 .523599"/>
+        <origin xyz="${wheel_offset_radius*sin(pi/3)} ${wheel_offset_radius*cos(pi/3)} 0.0" rpy="0 ${pi/2} ${pi/6}"/>
         <axis xyz="0 0 1"/>
     </joint>
@@ -76,5 +76,5 @@
         <parent link="base_link"/>
         <child link="wheel3"/>
-        <origin xyz="${wheel_offset_radius} 0.0 0.0" rpy="1.57 0 -.523599"/>
+        <origin xyz="${-wheel_offset_radius*sin(pi/3)} ${wheel_offset_radius*cos(pi/3)} 0.0" rpy="0 ${-pi/2} ${-pi/6}"/>
         <axis xyz="0 0 1"/>
     </joint>
@@ -97,7 +97,7 @@
         <parent link="base_link"/>
         <child link="paddle"/>
-        <origin xyz="0.0 0.0 ${chassis_height - wheel_radius}" rpy="0 0 1.57"/>
+        <origin xyz="0.0 0.0 ${origin_to_chassis_top}" rpy="0 0 ${pi}"/>
     </joint>
-    <link name="base_link">
+    <link name="paddle">
         <visual>
             <origin xyz="0.0 0.0 ${paddle_origin_offset}" rpy="0 0 0"/>

Commit message: Updated urdf and rviz config to match frames used for kinematics and odometry

File: pingpongbot_description/urdf/pingpongbot.urdf.xacro (robot description, xacro)
@@ -18,5 +18,5 @@
     <link name="base_link">
         <visual>
-            <origin xyz="0.0 0.0 0.0" rpy="0 0 0"/>
+            <origin xyz="0.0 0.0 0.0" rpy="0 0 ${pi}"/>
             <geometry>
                 <mesh filename="package://pingpongbot_description/meshes/chassis.stl" scale="1.0 1.0 1.0"/>
@@ -34,5 +34,5 @@
         <parent link="base_link"/>
         <child link="wheel1"/>
-        <origin xyz="0.0 ${-wheel_offset_radius} 0.0" rpy="${pi/2} 0 0"/>
+        <origin xyz="0.0 ${wheel_offset_radius} 0.0" rpy="${pi/2} 0 ${pi}"/>
         <axis xyz="0 0 1"/>
     </joint>
@@ -55,5 +55,5 @@
         <parent link="base_link"/>
         <child link="wheel2"/>
-        <origin xyz="${wheel_offset_radius*sin(pi/3)} ${wheel_offset_radius*cos(pi/3)} 0.0" rpy="0 ${pi/2} ${pi/6}"/>
+        <origin xyz="${wheel_offset_radius*sin(pi/3)} ${-wheel_offset_radius*cos(pi/3)} 0.0" rpy="${pi/2} 0 ${pi/3}"/>
         <axis xyz="0 0 1"/>
     </joint>
@@ -76,5 +76,5 @@
         <parent link="base_link"/>
         <child link="wheel3"/>
-        <origin xyz="${-wheel_offset_radius*sin(pi/3)} ${wheel_offset_radius*cos(pi/3)} 0.0" rpy="0 ${-pi/2} ${-pi/6}"/>
+        <origin xyz="${-wheel_offset_radius*sin(pi/3)} ${-wheel_offset_radius*cos(pi/3)} 0.0" rpy="${pi/2} 0 ${-pi/3}"/>
         <axis xyz="0 0 1"/>
     </joint>
@@ -97,5 +97,5 @@
         <parent link="base_link"/>
         <child link="paddle"/>
-        <origin xyz="0.0 0.0 ${origin_to_chassis_top}" rpy="0 0 ${pi}"/>
+        <origin xyz="0.0 0.0 ${origin_to_chassis_top}" rpy="0 0 0"/>
     </joint>
     <link name="paddle">

Commit message: current movement code - getting better

File: pingpongbot_description/urdf/pingpongbot.urdf.xacro (robot description, xacro)
@@ -10,13 +10,13 @@
         <color rgba="1 1 1 1"/>
     </material>
-    <link name="base_footprint"/>
+    <!-- <link name="base_footprint"/>
     <joint name="base_joint" type="fixed">
         <parent link="base_footprint"/>
         <child link="base_link"/>
         <origin xyz="0.0 0.0 ${wheel_radius}" rpy="0 0 0"/>
-    </joint>
+    </joint> -->
     <link name="base_link">
         <visual>
-            <origin xyz="0.0 0.0 0.0" rpy="0 0 ${pi}"/>
+            <origin xyz="0.0 0.0 ${wheel_radius}" rpy="0 0 ${pi}"/>
             <geometry>
                 <mesh filename="package://pingpongbot_description/meshes/chassis.stl" scale="1.0 1.0 1.0"/>
@@ -39,5 +39,5 @@
     <link name="wheel1">
         <visual>
-            <origin xyz="0.0 0.0 0.0" rpy="0 0 0"/>
+            <origin xyz="0.0 ${wheel_radius} 0.0" rpy="0 0 0"/>
             <geometry>
                 <mesh filename="package://pingpongbot_description/meshes/omniwheel.stl" scale="1.0 1.0 1.0"/>
@@ -60,5 +60,5 @@
     <link name="wheel2">
         <visual>
-            <origin xyz="0.0 0.0 0.0" rpy="0 0 0"/>
+            <origin xyz="0.0 ${wheel_radius} 0.0" rpy="0 0 0"/>
             <geometry>
                 <mesh filename="package://pingpongbot_description/meshes/omniwheel.stl" scale="1.0 1.0 1.0"/>
@@ -81,5 +81,5 @@
     <link name="wheel3">
         <visual>
-            <origin xyz="0.0 0.0 0.0" rpy="0 0 0"/>
+            <origin xyz="0.0 ${wheel_radius} 0.0" rpy="0 0 0"/>
             <geometry>
                 <mesh filename="package://pingpongbot_description/meshes/omniwheel.stl" scale="1.0 1.0 1.0"/>

Commit message: current code used for demo - still needs work/cleaning

File: pingpongbot_description/urdf/pingpongbot.urdf.xacro (robot description, xacro)
@@ -10,13 +10,7 @@
         <color rgba="1 1 1 1"/>
     </material>
-    <!-- <link name="base_footprint"/>
-    <joint name="base_joint" type="fixed">
-        <parent link="base_footprint"/>
-        <child link="base_link"/>
-        <origin xyz="0.0 0.0 ${wheel_radius}" rpy="0 0 0"/>
-    </joint> -->
     <link name="base_link">
         <visual>
-            <origin xyz="0.0 0.0 ${wheel_radius}" rpy="0 0 ${pi}"/>
+            <origin xyz="0.0 0.0 0.0" rpy="0 0 ${pi}"/>
             <geometry>
                 <mesh filename="package://pingpongbot_description/meshes/chassis.stl" scale="1.0 1.0 1.0"/>
@@ -31,4 +25,10 @@
         </collision>
     </link>
+    <link name="base_footprint"/>
+    <joint name="base_joint" type="fixed">
+        <parent link="base_link"/>
+        <child link="base_footprint"/>
+        <origin xyz="0.0 0.0 ${-wheel_radius}" rpy="0 0 0"/>
+    </joint>
     <joint name="wheel1_joint" type="continuous">
         <parent link="base_link"/>
@@ -39,5 +39,5 @@
     <link name="wheel1">
         <visual>
-            <origin xyz="0.0 ${wheel_radius} 0.0" rpy="0 0 0"/>
+            <origin xyz="0.0 0.0 0.0" rpy="0 0 0"/>
             <geometry>
                 <mesh filename="package://pingpongbot_description/meshes/omniwheel.stl" scale="1.0 1.0 1.0"/>
@@ -60,5 +60,5 @@
     <link name="wheel2">
         <visual>
-            <origin xyz="0.0 ${wheel_radius} 0.0" rpy="0 0 0"/>
+            <origin xyz="0.0 0.0 0.0" rpy="0 0 0"/>
             <geometry>
                 <mesh filename="package://pingpongbot_description/meshes/omniwheel.stl" scale="1.0 1.0 1.0"/>
@@ -81,5 +81,5 @@
     <link name="wheel3">
         <visual>
-            <origin xyz="0.0 ${wheel_radius} 0.0" rpy="0 0 0"/>
+            <origin xyz="0.0 0.0 0.0" rpy="0 0 0"/>
             <geometry>
                 <mesh filename="package://pingpongbot_description/meshes/omniwheel.stl" scale="1.0 1.0 1.0"/>
